File: SATA-backplane-10-inch-rack/SATA-backplane-10-inch-rack.kicad_pcb (KiCad board)
At the start: 2 copper layers, 210.1 x 69.6 mm, 41 parts, among them J101 Conn_01x06, J201 67800-5001, J202 1735284-2, J301 67800-5001, J302 1735284-2, J401 67800-5001, J402 1735284-2, J501 67800-5001, J502 1735284-2, J601 67800-5001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

Commit message: Fiddling with layout
Parts:
- removed H1, H2, H3, H4, H5, H6: MountingHole, MountingHole:MountingHole_3.7mm
- added JP102: SolderJumper, Jumper:SolderJumper-2_P1.3mm_Open_RoundedPad1.0x1.5mm, F.Cu at (193.2, 43.3)
- added U1: NCP1117-3.3_SOT223, Package_TO_SOT_SMD:SOT-223-3_TabPin2, F.Cu at (195.9, 37.4)
- D104: footprint LED_SMD:LED_0805_2012Metric_Pad1.15x1.40mm_HandSolder -> LED_SMD:LED_1206_3216Metric_Pad1.42x1.75mm_HandSolder
- D201, D301, D401, D501, D601, D701: footprint Package_TO_SOT_SMD:SOT-23 -> Package_TO_SOT_SMD:SOT-23_Handsoldering
- Q101, Q102: footprint Package_TO_SOT_SMD:SOT-323_SC-70 -> Package_TO_SOT_SMD:SOT-323_SC-70_Handsoldering
- moved C101 58.9 mm to (198.1, 80.6)
- moved C102 58.9 mm to (196.9, 71.4)
- moved C103 58.9 mm to (195.6, 62.3)
- moved D101 58.9 mm to (199.2, 75.7)
- moved D102 58.9 mm to (199.2, 68.1)
- moved D103 58.9 mm to (199.2, 60.5)
- moved J101 58.9 mm to (179.8, 62.4)
- moved C104 55.1 mm to (166.6, 36.1)
- moved JP101 55.1 mm to (172.4, 31.0)
- moved R101 55.1 mm to (168.6, 31.2)
- moved Q101 51.1 mm to (133.7, 45.2)
- moved R103 51.1 mm to (135.3, 38.6)
- moved R104 51.1 mm to (133.3, 38.6)
- moved Q102 51.1 mm to (134.1, 41.9)
- moved R105 51.1 mm to (133.4, 34.0)
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Routing:
- net /Port_5/STA/ACT: track 17.6 -> 4.66 mm, vias 4 -> 1
- net /Port_6/STA/ACT: track 28.9 -> 29.9 mm
- net /Port_4/STA/ACT: track 3.63 -> 4.66 mm
- net /Port_3/STA/ACT: track 3.63 -> 4.66 mm
- net /Port_2/STA/ACT: track 3.63 -> 4.66 mm
- net /Port_1/STA/ACT: track 3.63 -> 4.66 mm
- net Net-(D104-A): track 12.3 -> 13.1 mm
Other:
- outline, holes or cut-outs redrawn
- board text removed: "GND/black +12V/yellow GND/black +5V/red GND/black +3.3V/orange"
