File: SATA-backplane-10-inch-rack/Port.kicad_sch (KiCad schematic)
At the start: 3 parts, among them J201 67800-5001, J202 1735284-2

Commit message: Rearrange reference designators numbering and silkscreen items
Parts:
- renumbered D201 to D101, J201 to J101, J202 to J102
